File: hw/peripherals-board-v2/peripherals-board-v2.kicad_sch (KiCad schematic)
At the start: 26 parts, among them J1 Screw_Terminal_01x04, J10 Extra Servo, J10 RF24, J11 Conn_01x03, J12 Conn_01x03, J13 Conn_01x03, J13 RPLidar Motor, J2 Conn_01x04_Socket, J3 Conn_01x04_Socket, J4 Conn_01x04_Socket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

Commit message: Attempt to rescue schematic
Parts:
- removed J10: Extra Servo, Connector_PinHeader_2.54mm:PinHeader_1x03_P2.54mm_Vertical, symbol Connector:Conn_01x03_Pin
- removed J13: RPLidar Motor, symbol Connector:Conn_01x03_Socket
- renumbered J5 to #PWR037
Connections:
- net SPI1_SCK: now also J10.6 (Pin_6)
Other:
- note removed: "I2C Addresses: MPU6050: 0x68, 0x69 BMP085: 0x77 HMC5883L: 0x1E SSD1306 0x3C, 0x3D TFLuna: 0x07-0x77 BNO055: 0x28, 0x29 M24M02: 0x50-0x57"
- note removed: "IMU"
- note removed: "Motor Driver"
- note removed: "Power Supply"
